Commit message: Modify MJCF for matching with URDF

File: urdf/3D_Quad.urdf (robot description, URDF)
Before this commit: robot 3D_Quad, 24 links, 23 joints
Joints:
- joint FLHAA: axis 0 0 -1 -> 0 0 1
- joint FRHAA: axis 0 0 -1 -> 0 0 1
- joint RLHAA: axis 0 0 -1 -> 0 0 1
- joint RRHAA: axis 0 0 -1 -> 0 0 1

Commit message: urdf and xml are modified for match the coordinate

File: urdf/3D_Quad.urdf (robot description, URDF)
Before this commit: robot 3D_Quad, 24 links, 23 joints
Links:
- removed link torso_back_link
- link torso_front_link: mass 0.5 -> 1.4
Joints:
- removed joint torso_front_to_torso_back_joint
- joint FLHAA: axis 0 0 1 -> 1 0 0; origin xyz=0.2 0.15 0 rpy=0 1.5708 0 -> xyz=0.2 0.15 0 rpy=0 0 0
- joint FLHAA_point_fixed: origin xyz=0.2 0.15 0 rpy=3.14159 0 0 -> xyz=0.2 0.15 0 rpy=0 0 0
- joint FLHIP: origin xyz=0 0 0 rpy=0 0 0 -> xyz=0 0 0 rpy=0 1.5708 0
- joint FRHAA: axis 0 0 1 -> 1 0 0; origin xyz=0.2 -0.15 0 rpy=0 1.5708 0 -> xyz=0.2 -0.15 0 rpy=0 0 0
- joint FRHAA_point_fixed: origin xyz=0.2 -0.15 0 rpy=3.14159 0 0 -> xyz=0.2 -0.15 0 rpy=0 0 0
- joint FRHIP: origin xyz=0 0 0 rpy=0 0 0 -> xyz=0 0 0 rpy=0 1.5708 0
- joint FR_foot_joint: origin xyz=0 0 -0.25 rpy=0 0 0 -> xyz=0 0 -0.25 rpy=3.14159 0 0
- joint RLHAA: axis 0 0 1 -> 1 0 0; origin xyz=-0.2 0.15 0 rpy=0 1.5708 0 -> xyz=-0.2 0.15 0 rpy=0 0 0; parent torso_back_link -> torso_front_link
- joint RLHAA_point_fixed: origin xyz=-0.2 0.15 0 rpy=3.14159 0 0 -> xyz=-0.2 0.15 0 rpy=0 0 0; parent torso_back_link -> torso_front_link
- joint RLHIP: origin xyz=0 0 0 rpy=0 0 0 -> xyz=0 0 0 rpy=0 1.5708 0
- joint RL_foot_joint: origin xyz=0 0 -0.25 rpy=0 0 0 -> xyz=0 0 -0.25 rpy=3.14159 0 0
- joint RRHAA: axis 0 0 1 -> 1 0 0; origin xyz=-0.2 -0.15 0 rpy=0 1.5708 0 -> xyz=-0.2 -0.15 0 rpy=0 0 0; parent torso_back_link -> torso_front_link
- joint RRHAA_point_fixed: origin xyz=-0.2 -0.15 0 rpy=3.14159 0 0 -> xyz=-0.2 -0.15 0 rpy=0 0 0; parent torso_back_link -> torso_front_link
- joint RRHIP: origin xyz=0 0 0 rpy=0 0 0 -> xyz=0 0 0 rpy=0 1.5708 0
- joint RR_foot_joint: origin xyz=0 0 -0.25 rpy=0 0 0 -> xyz=0 0 -0.25 rpy=3.14159 0 0
- joint imu_joint: origin xyz=0 0 0 rpy=3.14159 0 0 -> xyz=0 0 0 rpy=0 0 0
- joint world_to_torso_front_joint: type fixed -> floating

Commit message: Add Crocoddyl Functions

File: urdf/3D_Quad.urdf (robot description, URDF)
Before this commit: robot 3D_Quad, 23 links, 22 joints
Joints:
- removed joint world_to_torso_front_joint
- added joint root_joint: type floating, parent root, child torso_front_link, origin xyz=0 0 0.375 rpy=0 0 0
